File: _autosave-pcb.kicad_pcb (KiCad board)
At the start: 2 copper layers, 24 parts, among them SW1 SW_Push, U1 ATmega32U4-AU, Y1 Crystal_GND24_Small

Commit message: peepeepoopooo
Parts:
- moved USB1 74.0 mm to (122.2, 136.5), turned to 270 degrees
- moved MX2 1.24 mm to (169.1, 163.5)
- moved MX3 1.15 mm to (188.1, 163.5)
- moved D2 1.12 mm to (177.0, 163.5)
- moved D3 1.12 mm to (196.1, 163.5)
- moved D1 0.79 mm to (177.0, 144.5)
- moved D4 0.79 mm to (196.1, 144.5)
- moved MX1 0.67 mm to (169.1, 144.4)
- moved MX4 0.48 mm to (188.1, 144.4)
- turned R1 to 270 degrees
Other:
- board outline added: 82.1 x 38.4 mm
Changed lines of the file:
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@@
   (general
     (thickness 1.6)
-    (drawings 0)
+    (drawings 8)
     (tracks 0)
     (zones 0)
@@
   )
   (module random-keyboard-parts:Molex-0548190589 (layer F.Cu)
-    (at 178.58125 88.60325)
-    (attr smd)
-    (fp_text reference USB1 (at 2.032 0 90) (layer F.SilkS)
-      (effects (font (size 1 1) (thickness 0.15)))
-    )
-    (fp_text value Molex-0548190589 (at -5.08 0 90) (layer Dwgs.User)
-      (effects (font (size 1 1) (thickness 0.15)))
-    )
-    (fp_text user %R (at 2 0 90) (layer F.CrtYd)
+    (at 122.2375 136.525 270)
+    (attr smd)
+    (fp_text reference USB1 (at 2.032 0) (layer F.SilkS)
+      (effects (font (size 1 1) (thickness 0.15)))
+    )
+    (fp_text value Molex-0548190589 (at -5.08 0) (layer Dwgs.User)
+      (effects (font (size 1 1) (thickness 0.15)))
+    )
+    (fp_text user %R (at 2 0) (layer F.CrtYd)
       (effects (font (size 1 1) (thickness 0.15)))
     )
@@
     (fp_line (start -1.75 -4.572) (end -1.75 4.572) (layer Dwgs.User) (width 0.15))
     (fp_line (start -3.75 -3.85) (end -3.75 3.85) (layer Dwgs.User) (width 0.15))
-    (pad 6 thru_hole oval (at 0 -3.65) (size 2.7 1.7) (drill oval 1.9 0.7) (layers *.Cu *.Mask)
+    (pad 6 thru_hole oval (at 0 -3.65 270) (size 2.7 1.7) (drill oval 1.9 0.7) (layers *.Cu *.Mask)
       (net 47 "Net-(USB1-Pad6)"))
-    (pad 6 thru_hole oval (at 0 3.65) (size 2.7 1.7) (drill oval 1.9 0.7) (layers *.Cu *.Mask)
+    (pad 6 thru_hole oval (at 0 3.65 270) (size 2.7 1.7) (drill oval 1.9 0.7) (layers *.Cu *.Mask)
       (net 47 "Net-(USB1-Pad6)"))
-    (pad 6 thru_hole oval (at 4.5 3.65) (size 2.7 1.7) (drill oval 1.9 0.7) (layers *.Cu *.Mask)
+    (pad 6 thru_hole oval (at 4.5 3.65 270) (size 2.7 1.7) (drill oval 1.9 0.7) (layers *.Cu *.Mask)
       (net 47 "Net-(USB1-Pad6)"))
-    (pad 6 thru_hole oval (at 4.5 -3.65) (size 2.7 1.7) (drill oval 1.9 0.7) (layers *.Cu *.Mask)
+    (pad 6 thru_hole oval (at 4.5 -3.65 270) (size 2.7 1.7) (drill oval 1.9 0.7) (layers *.Cu *.Mask)
       (net 47 "Net-(USB1-Pad6)"))
-    (pad 5 smd rect (at 4.5 -1.6) (size 2.25 0.5) (layers F.Cu F.Paste F.Mask)
+    (pad 5 smd rect (at 4.5 -1.6 270) (size 2.25 0.5) (layers F.Cu F.Paste F.Mask)
       (net 12 VCC))
-    (pad 4 smd rect (at 4.5 -0.8) (size 2.25 0.5) (layers F.Cu F.Paste F.Mask)
+    (pad 4 smd rect (at 4.5 -0.8 270) (size 2.25 0.5) (layers F.Cu F.Paste F.Mask)
       (net 15 D-))
-    (pad 3 smd rect (at 4.5 0) (size 2.25 0.5) (layers F.Cu F.Paste F.Mask)
+    (pad 3 smd rect (at 4.5 0 270) (size 2.25 0.5) (layers F.Cu F.Paste F.Mask)
       (net 17 D+))
-    (pad 2 smd rect (at 4.5 0.8) (size 2.25 0.5) (layers F.Cu F.Paste F.Mask)
+    (pad 2 smd rect (at 4.5 0.8 270) (size 2.25 0.5) (layers F.Cu F.Paste F.Mask)
       (net 48 "Net-(USB1-Pad2)"))
-    (pad 1 smd rect (at 4.5 1.6) (size 2.25 0.5) (layers F.Cu F.Paste F.Mask)
+    (pad 1 smd rect (at 4.5 1.6 270) (size 2.25 0.5) (layers F.Cu F.Paste F.Mask)
       (net 1 GND))
   )
@@
   )
   (module Resistor_SMD:R_0805_2012Metric (layer B.Cu)
-    (at 129.38125 150.01875 90)
+    (at 129.38125 150.01875 270)
     (descr "Resistor SMD 0805 (2012 Metric), square (rectangular) end terminal, IPC_7351 nominal, (Body size source: https://docs.google.com/spreadsheets/d/1BsfQQcO9C6DZCsRaXUlFlo91Tg2WpOkGARC1WS5S8t0/edit?usp=sharing), generated with kicad-footprint-generator")
     (tags resistor)
@@
     (fp_line (start -1 0.6) (end 1 0.6) (layer B.Fab) (width 0.1))
     (fp_line (start -1 -0.6) (end -1 0.6) (layer B.Fab) (width 0.1))
-    (pad 2 smd roundrect (at 0.9375 0 90) (size 0.975 1.4) (layers B.Cu B.Paste B.Mask) (roundrect_rratio 0.25)
+    (pad 2 smd roundrect (at 0.9375 0 270) (size 0.975 1.4) (layers B.Cu B.Paste B.Mask) (roundrect_rratio 0.25)
       (net 15 D-))
-    (pad 1 smd roundrect (at -0.9375 0 90) (size 0.975 1.4) (layers B.Cu B.Paste B.Mask) (roundrect_rratio 0.25)
+    (pad 1 smd roundrect (at -0.9375 0 270) (size 0.975 1.4) (layers B.Cu B.Paste B.Mask) (roundrect_rratio 0.25)
       (net 16 "Net-(R1-Pad1)"))
     (model ${KISYS3DMOD}/Resistor_SMD.3dshapes/R_0805_2012Metric.wrl
@@
   )
   (module MX_Alps_Hybrid:MX-1U (layer F.Cu)
-    (at 188.6 144.35625)
+    (at 188.11875 144.35625)
     (fp_text reference MX4 (at 0 3.175) (layer Dwgs.User)
       (effects (font (size 1 1) (thickness 0.15)))
@@
   )
   (module MX_Alps_Hybrid:MX-1U (layer F.Cu)
-    (at 188.6 164.55625)
+    (at 188.11875 163.5125)
     (fp_text reference MX3 (at 0 3.175) (layer Dwgs.User)
       (effects (font (size 1 1) (thickness 0.15)))
@@
   )
   (module MX_Alps_Hybrid:MX-1U (layer F.Cu)
-    (at 168.4 164.55625)
+    (at 169.06875 163.5125)
     (fp_text reference MX2 (at 0 3.175) (layer Dwgs.User)
       (effects (font (size 1 1) (thickness 0.15)))
@@
   )
   (module MX_Alps_Hybrid:MX-1U (layer F.Cu)
-    (at 168.4 144.35625)
+    (at 169.06875 144.35625)
     (fp_text reference MX1 (at 0 3.175) (layer Dwgs.User)
       (effects (font (size 1 1) (thickness 0.15)))
@@
   )
   (module Diode_SMD:D_SOD-123 (layer B.Cu)
-    (at 196.85 144.4625 90)
+    (at 196.05625 144.4625 90)
     (descr SOD-123)
     (tags SOD-123)
@@
   )
   (module Diode_SMD:D_SOD-123 (layer B.Cu)
-    (at 196.85 164.30625 90)
+    (at 196.05625 163.5125 90)
     (descr SOD-123)
     (tags SOD-123)
@@
   )
   (module Diode_SMD:D_SOD-123 (layer B.Cu)
-    (at 176.2125 164.30625 90)
+    (at 177.00625 163.5125 90)
     (descr SOD-123)
     (tags SOD-123)
@@
   )
   (module Diode_SMD:D_SOD-123 (layer B.Cu)
-    (at 176.2125 144.4625 90)
+    (at 177.00625 144.4625 90)
     (descr SOD-123)
     (tags SOD-123)
@@
     )
   )
+  (gr_line (start 195.2625 134.77875) (end 117.95125 134.71525) (layer Edge.Cuts) (width 0.25))
+  (gr_arc (start 117.95125 137.0965) (end 117.95125 134.71525) (angle -90) (layer Edge.Cuts) (width 0.25))
+  (gr_line (start 115.57 137.0965) (end 115.53825 170.6245) (layer Edge.Cuts) (width 0.25))
+  (gr_arc (start 117.9195 170.6245) (end 117.9195 173.00575) (angle 90) (layer Edge.Cuts) (width 0.25))
+  (gr_line (start 195.23075 173.06925) (end 117.9195 173.00575) (layer Edge.Cuts) (width 0.25))
+  (gr_line (start 197.64375 137.16) (end 197.612 170.688) (layer Edge.Cuts) (width 0.25))
+  (gr_arc (start 195.23075 170.688) (end 197.612 170.688) (angle 90) (layer Edge.Cuts) (width 0.25))
+  (gr_arc (start 195.2625 137.16) (end 197.64375 137.16) (angle -90) (layer Edge.Cuts) (width 0.25))
 )
