File: pcb.kicad_pcb (KiCad board)
At the start: 2 copper layers, 24 parts, among them SW1 SW_Push, U1 ATmega32U4-AU, Y1 Crystal_GND24_Small

Commit message: yep
Parts:
- F1, R2, R3, R4, SW1, USB1: moved to B.Cu
- moved USB1 71.4 mm to (107.2, 88.1), turned to 270 degrees
- moved R2 70.7 mm to (108.0, 100.8), turned to 90 degrees
- moved SW1 61.7 mm to (106.4, 121.4), turned to 180 degrees
- moved C6 61.1 mm to (115.1, 112.7)
- moved R3 60.9 mm to (115.1, 101.6), turned to 90 degrees
- moved F1 59.6 mm to (103.2, 104.8), turned to 90 degrees
- moved C4 55.6 mm to (119.1, 96.0), turned to 270 degrees
- moved R1 54.7 mm to (105.6, 100.8)
- moved Y1 52.0 mm to (123.8, 96.0)
- moved MX3 51.9 mm to (173.0, 115.1)
- moved D3 51.7 mm to (181.0, 115.1)
- moved MX2 51.5 mm to (154.0, 115.1)
- moved D2 51.2 mm to (161.9, 115.1)
- moved D4 51.0 mm to (181.0, 96.0)
- moved MX4 50.9 mm to (173.0, 95.9)
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Connections:
- U1 pad 16: Net-(C4-Pad1) -> Net-(U1-Pad16)
- U1 pad 26: Net-(U1-Pad26) -> COL0
- U1 pad 27: Net-(U1-Pad27) -> COL1
- U1 pad 28: Net-(U1-Pad28) -> ROW0
- U1 pad 29: Net-(U1-Pad29) -> ROW1
Routing:
- net GND: track 0.00 -> 106.6 mm
- net +5V: track 0.00 -> 79.3 mm, vias 0 -> 7
- net ROW0: track 0.00 -> 76.4 mm
- net ROW1: track 0.00 -> 63.0 mm, vias 0 -> 2
- net COL1: track 0.00 -> 60.0 mm
- net COL0: track 0.00 -> 42.2 mm, vias 0 -> 3
- net Net-(R3-Pad2): track 0.00 -> 32.5 mm, vias 0 -> 2
- net Net-(C3-Pad1): track 0.00 -> 23.7 mm, vias 0 -> 3
- net Net-(C4-Pad1): track 0.00 -> 23.7 mm
- net Net-(R1-Pad1): track 0.00 -> 22.3 mm
- net Net-(R2-Pad1): track 0.00 -> 20.7 mm
- net VCC: track 0.00 -> 11.7 mm
- net Net-(C6-Pad1): track 0.00 -> 8.31 mm, vias 0 -> 2
- net D+: track 0.00 -> 7.59 mm
- net D-: track 0.00 -> 7.59 mm
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Other:
- board outline added: 82.1 x 38.4 mm
- net class Default: trace_width 0.25 -> 0.254
- net class power added: clearance 0.2, trace_width 0.381, via_dia 0.8, via_drill 0.4
